File: hardware/_autosave-inputs.kicad_sch (KiCad schematic)
At the start: 15 parts, among them J2 CLK_IN, J3 RST_IN, J4 SCENE_CV

Commit message: Complete hierarchical schematic sheets and fix wiring
- Complete encoder_leds sheet with MAX7219 + 64 LEDs
- Complete ui_leds sheet with MAX7219 + 45 LEDs
- Complete buttons sheet with MCP23017 + 40 buttons
- Complete display sheet with OLED I2C connector
- Complete pots sheet with 3 potentiometers
- Complete encoders sheet with 8 rotary encoders on MCP23017
- Fix inputs sheet hierarchical labels (CLK_IN, RST_IN, SCENE_CV_IN)
- Update MCU sheet with ADC hierarchical labels
- Update root sheet with hierarchical pin connections
- Various ERC fixes and wiring corrections

Co-Authored-By: Claude Opus 4.5 <noreply@anthropic.com>
Parts:
- J2, J3, J4: footprint (none) -> Connector_Audio:Jack_3.5mm_QingPu_WQP-PJ398SM_Vertical_CircularHoles
- R1, R2, R3, R4, R5, R6: footprint (none) -> Resistor_SMD:R_0201_0603Metric_Pad0.64x0.40mm_HandSolder
Changed lines of the file:
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@@
 			)
 		)
-		(property "Footprint" ""
+		(property "Footprint" "Resistor_SMD:R_0201_0603Metric_Pad0.64x0.40mm_HandSolder"
 			(at 63.5 61.468 90)
 			(effects
@@
 			)
 		)
-		(property "Footprint" ""
+		(property "Footprint" "Connector_Audio:Jack_3.5mm_QingPu_WQP-PJ398SM_Vertical_CircularHoles"
 			(at 29.21 59.69 0)
 			(effects
@@
 			)
 		)
-		(property "Footprint" ""
+		(property "Footprint" "Connector_Audio:Jack_3.5mm_QingPu_WQP-PJ398SM_Vertical_CircularHoles"
 			(at 30.48 143.51 0)
 			(effects
@@
 			)
 		)
-		(property "Footprint" ""
+		(property "Footprint" "Resistor_SMD:R_0201_0603Metric_Pad0.64x0.40mm_HandSolder"
 			(at 79.502 151.13 90)
 			(effects
@@
 			)
 		)
-		(property "Footprint" ""
+		(property "Footprint" "Resistor_SMD:R_0201_0603Metric_Pad0.64x0.40mm_HandSolder"
 			(at 78.232 67.31 90)
 			(effects
@@
 			)
 		)
-		(property "Footprint" ""
+		(property "Footprint" "Resistor_SMD:R_0201_0603Metric_Pad0.64x0.40mm_HandSolder"
 			(at 64.77 145.288 90)
 			(effects
@@
 			)
 		)
-		(property "Footprint" ""
+		(property "Footprint" "Connector_Audio:Jack_3.5mm_QingPu_WQP-PJ398SM_Vertical_CircularHoles"
 			(at 30.48 100.33 0)
 			(effects
@@
 			)
 		)
-		(property "Footprint" ""
+		(property "Footprint" "Resistor_SMD:R_0201_0603Metric_Pad0.64x0.40mm_HandSolder"
 			(at 78.232 107.95 90)
 			(effects
@@
 			)
 		)
-		(property "Footprint" ""
+		(property "Footprint" "Resistor_SMD:R_0201_0603Metric_Pad0.64x0.40mm_HandSolder"
 			(at 63.5 102.108 90)
 			(effects
