File: hardware/_autosave-mcu.kicad_sch (KiCad schematic)
At the start: 14 parts, among them J5 Conn_01x04, SW9 SW_Push, U3 STM32G431C6Tx, Y1 8MHz

Commit message: Complete hierarchical schematic sheets and fix wiring
- Complete encoder_leds sheet with MAX7219 + 64 LEDs
- Complete ui_leds sheet with MAX7219 + 45 LEDs
- Complete buttons sheet with MCP23017 + 40 buttons
- Complete display sheet with OLED I2C connector
- Complete pots sheet with 3 potentiometers
- Complete encoders sheet with 8 rotary encoders on MCP23017
- Fix inputs sheet hierarchical labels (CLK_IN, RST_IN, SCENE_CV_IN)
- Update MCU sheet with ADC hierarchical labels
- Update root sheet with hierarchical pin connections
- Various ERC fixes and wiring corrections

Co-Authored-By: Claude Opus 4.5 <noreply@anthropic.com>
Parts:
- J5: footprint (none) -> Connector_JST:JST_PH_B4B-PH-K_1x04_P2.00mm_Vertical
- R7, R8: footprint (none) -> Resistor_SMD:R_0201_0603Metric_Pad0.64x0.40mm_HandSolder
- SW9: footprint Button_Switch_SMD:SW_Push_1P1T_NO_CK_KSC7xxJ -> Button_Switch_THT:SW_PUSH_1P1T_6x3.5mm_H5.0_APEM_MJTP1250
- Y1: footprint (none) -> Crystal:Crystal_HC49-4H_Vertical
Changed lines of the file:
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@@
 			)
 		)
-		(property "Footprint" ""
+		(property "Footprint" "Connector_JST:JST_PH_B4B-PH-K_1x04_P2.00mm_Vertical"
 			(at 182.88 142.24 0)
 			(effects
@@
 			)
 		)
-		(property "Footprint" ""
+		(property "Footprint" "Resistor_SMD:R_0201_0603Metric_Pad0.64x0.40mm_HandSolder"
 			(at 115.57 124.968 90)
 			(effects
@@
 			)
 		)
-		(property "Footprint" "Button_Switch_SMD:SW_Push_1P1T_NO_CK_KSC7xxJ"
+		(property "Footprint" "Button_Switch_THT:SW_PUSH_1P1T_6x3.5mm_H5.0_APEM_MJTP1250"
 			(at 101.6 53.34 0)
 			(effects
@@
 			)
 		)
-		(property "Footprint" ""
+		(property "Footprint" "Resistor_SMD:R_0201_0603Metric_Pad0.64x0.40mm_HandSolder"
 			(at 85.852 58.42 90)
 			(effects
@@
 			)
 		)
-		(property "Footprint" ""
+		(property "Footprint" "Crystal:Crystal_HC49-4H_Vertical"
 			(at 105.41 80.01 0)
 			(effects
