File: hardware/sengbard.kicad_pcb (KiCad board)
At the start: 2 copper layers, 209 parts, among them J1 Eurorack_Power, J17 GATE_T1, J18 GATE_T2, J19 GATE_T3, J2 CLK_IN, J20 CLK_OUT, J21 RST_OUT, J3 RST_IN, J4 SCENE_CV, J5 SWD, J6 CV_OUT_T1, J7 CV_OUT_T3, J8 CV_OUT_T2, SW1 EC11, SW10 SW_Push, SW11 SW_Push, SW12 SW_Push, SW13 SW_Push, SW14 SW_Push, SW15 SW_Push, SW16 SW_Push, SW17 SW_Push, SW18 SW_Push, SW19 SW_Push, SW2 EC11, SW20 SW_Push, SW21 SW_Push, SW22 SW_Push, SW23 SW_Push, SW24 SW_Push, SW25 SW_Push, SW26 SW_Push, SW27 SW_Push, SW28 SW_Push, SW29 SW_Push, SW3 EC11, SW30 SW_Push, SW31 SW_Push, SW32 SW_Push, SW33 SW_Push, SW34 SW_Push, SW35 SW_Push, SW36 SW_Push, SW37 SW_Push, SW38 SW_Push, SW39 SW_Push, SW4 EC11, SW40 SW_Push, SW41 SW_Push, SW42 SW_Push, SW43 SW_Push, SW44 SW_Push, SW45 SW_Push, SW46 SW_Push, SW47 EC11, SW48 EC11, SW49 EC11, SW5 EC11, SW6 EC11, SW7 EC11, SW8 EC11, SW9 SW_Push, U1 MP1584 (3.3V), U2 MP1584 (5V), U3 STM32G431C6Tx, U4 MCP23017, U5 Opamp_Quad, U9 MCP23017_SP, Y1 8MHz

Commit message: Complete hierarchical schematic sheets and fix wiring
- Complete encoder_leds sheet with MAX7219 + 64 LEDs
- Complete ui_leds sheet with MAX7219 + 45 LEDs
- Complete buttons sheet with MCP23017 + 40 buttons
- Complete display sheet with OLED I2C connector
- Complete pots sheet with 3 potentiometers
- Complete encoders sheet with 8 rotary encoders on MCP23017
- Fix inputs sheet hierarchical labels (CLK_IN, RST_IN, SCENE_CV_IN)
- Update MCU sheet with ADC hierarchical labels
- Update root sheet with hierarchical pin connections
- Various ERC fixes and wiring corrections

Co-Authored-By: Claude Opus 4.5 <noreply@anthropic.com>
Parts:
- removed C1, C2, C3: 100uF, Capacitor_THT:CP_Radial_D8.0mm_P3.50mm
- removed C4, C5, C6: 100nF, Capacitor_SMD:C_0805_2012Metric
- removed C7, C8: 20pF, Capacitor_SMD:C_0603_1608Metric
- removed J17: GATE_T1, Connector_Audio:Jack_3.5mm_QingPu_WQP-PJ398SM_Vertical_CircularHoles
- removed J18: GATE_T2, Connector_Audio:Jack_3.5mm_QingPu_WQP-PJ398SM_Vertical_CircularHoles
- removed J19: GATE_T3, Connector_Audio:Jack_3.5mm_QingPu_WQP-PJ398SM_Vertical_CircularHoles
- removed J20: CLK_OUT, Connector_Audio:Jack_3.5mm_QingPu_WQP-PJ398SM_Vertical_CircularHoles
- removed J21: RST_OUT, Connector_Audio:Jack_3.5mm_QingPu_WQP-PJ398SM_Vertical_CircularHoles
- added FB1: FerriteBead, Inductor_SMD:L_Eaton_MCL2012V1, F.Cu at (211.8, 53.9)
- added J10: GATE_T1, Connector_Audio:Jack_3.5mm_QingPu_WQP-PJ398SM_Vertical_CircularHoles, F.Cu at (166.0, 88.9)
- added J11: GATE_T2, Connector_Audio:Jack_3.5mm_QingPu_WQP-PJ398SM_Vertical_CircularHoles, F.Cu at (177.0, 88.9)
- added J12: GATE_T3, Connector_Audio:Jack_3.5mm_QingPu_WQP-PJ398SM_Vertical_CircularHoles, F.Cu at (188.1, 88.9)
- added J13: CLK_OUT, Connector_Audio:Jack_3.5mm_QingPu_WQP-PJ398SM_Vertical_CircularHoles, F.Cu at (199.1, 88.9)
- added J14: RST_OUT, Connector_Audio:Jack_3.5mm_QingPu_WQP-PJ398SM_Vertical_CircularHoles, F.Cu at (210.2, 88.9)
- added J9: OLED, Connector_JST:JST_PH_B4B-PH-K_1x04_P2.00mm_Vertical, F.Cu at (186.4, 66.2)
- added L1: 10uH, Inductor_SMD:L_0201_0603Metric_Pad0.64x0.40mm_HandSolder, F.Cu at (211.1, 56.4)
- added R10: 27k, Resistor_SMD:R_0201_0603Metric_Pad0.64x0.40mm_HandSolder, F.Cu at (199.1, 82.3)
- added R16: 100R, Resistor_SMD:R_0201_0603Metric_Pad0.64x0.40mm_HandSolder, F.Cu at (161.9, 103.3)
- added R17: 100R, Resistor_SMD:R_0201_0603Metric_Pad0.64x0.40mm_HandSolder, F.Cu at (161.9, 105.1)
- added R18: 4.7k, Resistor_SMD:R_0201_0603Metric_Pad0.64x0.40mm_HandSolder, F.Cu at (161.9, 106.8)
- added R19: 100R, Resistor_SMD:R_0201_0603Metric_Pad0.64x0.40mm_HandSolder, F.Cu at (161.9, 108.6)
- added R20: 4.7k, Resistor_SMD:R_0201_0603Metric_Pad0.64x0.40mm_HandSolder, F.Cu at (161.9, 110.3)
- added R25: 4.7k, Resistor_SMD:R_0201_0603Metric_Pad0.64x0.40mm_HandSolder, F.Cu at (161.9, 112.1)
- added R26: 100R, Resistor_SMD:R_0201_0603Metric_Pad0.64x0.40mm_HandSolder, F.Cu at (164.7, 103.3)
- added R27: 4.7k, Resistor_SMD:R_0201_0603Metric_Pad0.64x0.40mm_HandSolder, F.Cu at (164.7, 105.1)
- added R28: 4.7k, Resistor_SMD:R_0201_0603Metric_Pad0.64x0.40mm_HandSolder, F.Cu at (164.7, 106.8)
- added R29: 100R, Resistor_SMD:R_0201_0603Metric_Pad0.64x0.40mm_HandSolder, F.Cu at (164.7, 108.6)
- added R30: 24.9k, Resistor_SMD:R_0201_0603Metric_Pad0.64x0.40mm_HandSolder, F.Cu at (211.1, 58.1)
- added R31: 100k, Resistor_SMD:R_0201_0603Metric_Pad0.64x0.40mm_HandSolder, F.Cu at (211.1, 59.9)
- added R7: 10k, Resistor_SMD:R_0201_0603Metric_Pad0.64x0.40mm_HandSolder, F.Cu at (210.1, 142.0)
- added R8: 10k, Resistor_SMD:R_0201_0603Metric_Pad0.64x0.40mm_HandSolder, F.Cu at (210.1, 143.8)
- added R9: 27k, Resistor_SMD:R_0201_0603Metric_Pad0.64x0.40mm_HandSolder, F.Cu at (180.0, 64.4)
- added RV1: 10k, Potentiometer_SMD:Potentiometer_ACP_CA6-VSMD_Vertical, F.Cu at (202.0, 119.0)
- added RV2: 10k, Potentiometer_SMD:Potentiometer_ACP_CA6-VSMD_Vertical, F.Cu at (202.0, 127.0)
- added RV3: 10k, Potentiometer_SMD:Potentiometer_ACP_CA6-VSMD_Vertical, F.Cu at (202.0, 135.1)
- D3, D4, D5: value BAT54 -> BAT54W; footprint Diode_SMD:D_SOD-123 -> Package_TO_SOT_SMD:SOT-323_SC-70
- J1: value Eurorack_Power -> Conn_02x05_Odd_Even
- J5: value SWD -> Conn_01x04; footprint Connector_PinHeader_2.54mm:PinHeader_1x04_P2.54mm_Vertical -> Connector_JST:JST_PH_B4B-PH-K_1x04_P2.00mm_Vertical
- R1, R2: value 100K -> 100k; footprint Resistor_SMD:R_0805_2012Metric -> Resistor_SMD:R_0201_0603Metric_Pad0.64x0.40mm_HandSolder
- R11, R23, R24: footprint Resistor_SMD:R_0805_2012Metric -> Resistor_SMD:R_0201_0603Metric_Pad0.64x0.40mm_HandSolder
- R12, R13: value 10K -> 10k; footprint Resistor_SMD:R_0805_2012Metric -> Resistor_SMD:R_0201_0603Metric_Pad0.64x0.40mm_HandSolder
- R14, R15, R21: value 20K -> 20k; footprint Resistor_SMD:R_0805_2012Metric -> Resistor_SMD:R_0201_0603Metric_Pad0.64x0.40mm_HandSolder
- R22: value 100 -> 100R; footprint Resistor_SMD:R_0805_2012Metric -> Resistor_SMD:R_0201_0603Metric_Pad0.64x0.40mm_HandSolder
- R3: value 68K -> 100k; footprint Resistor_SMD:R_0805_2012Metric -> Resistor_SMD:R_0201_0603Metric_Pad0.64x0.40mm_HandSolder
- R4, R5: value 47K -> 47k; footprint Resistor_SMD:R_0805_2012Metric -> Resistor_SMD:R_0201_0603Metric_Pad0.64x0.40mm_HandSolder
- R6: value 33K -> 47k; footprint Resistor_SMD:R_0805_2012Metric -> Resistor_SMD:R_0201_0603Metric_Pad0.64x0.40mm_HandSolder
- SW1, SW2, SW3, SW4, SW47, SW48, SW49, SW5, SW6, SW7, SW8: value EC11 -> RotaryEncoder; footprint Rotary_Encoder:RotaryEncoder_Alps_EC11E-Switch_Vertical_H20mm -> Rotary_Encoder:RotaryEncoder_Alps_EC12E_Vertical_H20mm_CircularMountingHoles
- SW10, SW11, SW12, SW13, SW14, SW15, SW16, SW17, SW18, SW19, SW20, SW21, SW22, SW23, SW24, SW25, SW26, SW27, SW28, SW29, SW30, SW31, SW32, SW33, SW34, SW35, SW36, SW37, SW38, SW39, SW40, SW41, SW42, SW43, SW44, SW45, SW46, SW9: footprint Button_Switch_SMD:SW_Push_1P1T_NO_CK_KSC7xxJ -> Button_Switch_THT:SW_PUSH_1P1T_6x3.5mm_H5.0_APEM_MJTP1250
- U1: value MP1584 (3.3V) -> TPS54202DDC; footprint Connector_PinHeader_2.54mm:PinHeader_1x04_P2.54mm_Vertical -> Package_TO_SOT_SMD:SOT-23-6
- U2: value MP1584 (5V) -> AP2112K-3.3; footprint Connector_PinHeader_2.54mm:PinHeader_1x04_P2.54mm_Vertical -> Package_TO_SOT_SMD:SOT-23-5
- U4: value MCP23017 -> MCP23017_SP
- moved SW47 205.1 mm to (134.9, 39.8), turned to 0 degrees
- moved SW48 194.1 mm to (134.9, 55.3), turned to 0 degrees
- moved SW49 187.5 mm to (134.9, 70.9), turned to 0 degrees
- moved SW41 175.1 mm to (124.7, 42.1)
- moved SW40 173.6 mm to (124.7, 37.0)
- moved SW33 169.5 mm to (114.4, 52.2)
- moved SW32 168.1 mm to (114.4, 47.1)
- moved SW31 166.6 mm to (114.4, 42.1)
- moved SW30 165.2 mm to (114.4, 37.0)
- moved SW25 164.4 mm to (104.1, 62.3)
- moved SW24 163.0 mm to (104.1, 57.2)
- moved SW23 161.7 mm to (104.1, 52.2)
- moved SW46 161.3 mm to (124.7, 67.3)
- moved SW22 160.4 mm to (104.1, 47.1)
- moved SW45 160.4 mm to (124.7, 62.3)
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Connections:
- D1 pad 1: /Power Supply/+12V_PROT -> +12V
- D1 pad 2: +12V -> Net-(D1-A)
- D2 pad 1: -12V -> -12V_IN
- D2 pad 2: GND -> -12V
- D3 pad 1: /CV Inputs/PA1 -> +3V3
- D3 pad 2: +3V3 -> unconnected-(D3-NC-Pad2)
- D4 pad 1: /CV Inputs/PA2 -> +3V3
- D4 pad 2: +3V3 -> unconnected-(D4-NC-Pad2)
- D5 pad 1: /CV Inputs/PA3 -> +3V3
- D5 pad 2: +3V3 -> unconnected-(D5-NC-Pad2)
- J1 pad 1: -12V -> -12V_IN
- J1 pad 10: +12V -> Net-(D1-A)
- J1 pad 2: -12V -> -12V_IN
- J1 pad 3: GND -> GND_IN
- J1 pad 4: GND -> GND_IN
- J1 pad 5: GND -> GND_IN
- J1 pad 6: GND -> GND_IN
- J1 pad 7: GND -> GND_IN
- J1 pad 8: GND -> GND_IN
- J1 pad 9: +12V -> +12V_IN
- J2 pad S: unconnected-(J2-PadS) -> GND
- J2 pad TN: GND -> (no net)
- J3 pad S: unconnected-(J3-PadS) -> GND
- J3 pad TN: GND -> (no net)
- J4 pad S: unconnected-(J4-PadS) -> GND
- J4 pad TN: GND -> (no net)
- J5 pad 1: unconnected-(J5-Pin_1-Pad1) -> +3V3
- J6 pad S: GND -> Net-(J6-PadS)
- J6 pad T: Net-(J6-PadT) -> GND
- J7 pad S: GND -> Net-(J7-PadS)
- J7 pad T: Net-(J7-PadT) -> GND
- J8 pad S: GND -> Net-(J8-PadS)
- J8 pad T: Net-(J8-PadT) -> GND
- R1 pad 2: /CV Inputs/PA1 -> /CV Inputs/CLK_IN
- R15 pad 1: Net-(U5B--) -> Net-(U5C--)
- R2 pad 2: /CV Inputs/PA2 -> /CV Inputs/RST_IN
- R21 pad 1: Net-(R21-Pad1) -> Net-(U5B--)
- R21 pad 2: Net-(U5C--) -> Net-(R21-Pad2)
- R22 pad 2: Net-(J6-PadT) -> Net-(J6-PadS)
- R23 pad 1: Net-(R21-Pad1) -> Net-(R15-Pad2)
- R23 pad 2: Net-(J7-PadT) -> Net-(J7-PadS)
- R24 pad 1: Net-(R15-Pad2) -> Net-(R21-Pad2)
- R24 pad 2: Net-(J8-PadT) -> Net-(J8-PadS)
- R3 pad 2: /CV Inputs/PA3 -> /CV Inputs/SCENE_CV_IN
- R4 pad 1: /CV Inputs/PA1 -> /CV Inputs/CLK_IN
- R5 pad 1: /CV Inputs/PA2 -> /CV Inputs/RST_IN
- R6 pad 1: /CV Inputs/PA3 -> /CV Inputs/SCENE_CV_IN
- SW1 pad A: Net-(U4-GPA0) -> Net-(U4-GPB0)
- SW1 pad B: Net-(U4-GPA1) -> Net-(U4-GPB1)
- SW2 pad A: Net-(U4-GPA2) -> Net-(U4-GPB2)
- SW2 pad B: Net-(U4-GPA3) -> Net-(U4-GPB3)
- SW3 pad A: Net-(U4-GPA4) -> Net-(U4-GPB4)
- SW3 pad B: Net-(U4-GPA5) -> Net-(U4-GPB5)
- SW4 pad A: Net-(U4-GPA6) -> Net-(U4-GPB6)
- SW4 pad B: Net-(U4-GPA7) -> Net-(U4-GPB7)
- SW5 pad A: Net-(U4-GPB0) -> Net-(U4-GPA0)
- SW5 pad B: Net-(U4-GPB1) -> Net-(U4-GPA1)
- SW6 pad A: Net-(U4-GPB2) -> Net-(U4-GPA2)
- SW6 pad B: Net-(U4-GPB3) -> Net-(U4-GPA3)
- SW7 pad A: Net-(U4-GPB4) -> Net-(U4-GPA4)
- SW7 pad B: Net-(U4-GPB5) -> Net-(U4-GPA5)
- SW8 pad A: Net-(U4-GPB6) -> Net-(U4-GPA6)
- SW8 pad B: Net-(U4-GPB7) -> Net-(U4-GPA7)
- U1 pad 1: /Power Supply/+12V_PROT -> GND
- U1 pad 2: GND -> Net-(U1-SW)
- U1 pad 3: +3V3 -> +12V
- U1 pad 4: GND -> Net-(U1-FB)
- U2 pad 1: /Power Supply/+12V_PROT -> +5V
- U2 pad 4: GND -> unconnected-(U2-NC-Pad4)
- U3 pad 1: unconnected-(U3-VBAT-Pad1) -> +3V3
- U3 pad 10: /MCU - STM32G431/RST_IN -> /CV Inputs/RST_IN
- U3 pad 11: /MCU - STM32G431/SCENE_CV_IN -> /CV Inputs/SCENE_CV_IN
- U3 pad 20: Net-(U3-VDDA) -> +3V3
- U3 pad 21: Net-(U3-VDDA) -> +3V3
- U3 pad 24: Net-(C12-Pad2) -> +3V3
- U3 pad 31: unconnected-(U3-PA9-Pad31) -> /MCU - STM32G431/ADC_BPM
- U3 pad 32: unconnected-(U3-PA10-Pad32) -> /MCU - STM32G431/ADC_SWG
- U3 pad 33: unconnected-(U3-PA11-Pad33) -> /MCU - STM32G431/ADC_PW
- U3 pad 36: Net-(C11-Pad2) -> +3V3
- U3 pad 48: Net-(C10-Pad2) -> +3V3
- U3 pad 9: /MCU - STM32G431/CLK_IN -> /CV Inputs/CLK_IN
- U5 pad 7: Net-(R15-Pad2) -> Net-(R21-Pad2)
- U5 pad 8: Net-(R21-Pad1) -> Net-(R15-Pad2)
Routing:
- net Net-(U3-PF0): track 11.7 -> 0.00 mm
- net Net-(U3-PF1): track 11.4 -> 0.00 mm
