File: hardware/display.kicad_sch (KiCad schematic)
At the start: 1 part, among them J9 OLED

Commit message: Complete hierarchical schematic sheets and fix wiring
- Complete encoder_leds sheet with MAX7219 + 64 LEDs
- Complete ui_leds sheet with MAX7219 + 45 LEDs
- Complete buttons sheet with MCP23017 + 40 buttons
- Complete display sheet with OLED I2C connector
- Complete pots sheet with 3 potentiometers
- Complete encoders sheet with 8 rotary encoders on MCP23017
- Fix inputs sheet hierarchical labels (CLK_IN, RST_IN, SCENE_CV_IN)
- Update MCU sheet with ADC hierarchical labels
- Update root sheet with hierarchical pin connections
- Various ERC fixes and wiring corrections

Co-Authored-By: Claude Opus 4.5 <noreply@anthropic.com>
Changed lines of the file:
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@@
 	)
 	(symbol
+		(lib_name "Conn_01x04_1")
 		(lib_id "Connector_Generic:Conn_01x04")
 		(at 154.94 93.98 0)
@@
 		(on_board yes)
 		(dnp no)
+		(fields_autoplaced yes)
 		(property "Reference" "J9"
-			(at 154.94 84.98 0)
+			(at 157.48 93.9799 0)
 			(effects
 				(font
 					(size 1.27 1.27)
 				)
+				(justify left)
 			)
 		)
 		(property "Value" "OLED"
-			(at 154.94 103.98 0)
+			(at 157.48 96.5199 0)
 			(effects
 				(font
 					(size 1.27 1.27)
 				)
+				(justify left)
 			)
 		)
@@
 			)
 		)
-		(property "Description" ""
+		(property "Description" "Generic connector, single row, 01x04, script generated (kicad-library-utils/schlib/autogen/connector/)"
 			(at 154.94 93.98 0)
 			(effects
@@
 					(size 1.27 1.27)
 				)
+				(hide yes)
 			)
+		)
+		(pin "4"
+		)
+		(pin "3"
+		)
+		(pin "2"
 		)
 		(pin "1"
 		)
-		(pin "2"
-		)
-		(pin "3"
-		)
-		(pin "4"
-		)
 		(instances
-			(project "sengbard"
+			(project ""
 				(path "/e1e5c1f0-1234-5678-9abc-def012345678/31fc420d-f921-43e0-8f58-c12b1db1de7b"
 					(reference "J9")

Commit message: Assign footprints to all schematic components
SMD footprints assigned:
- Capacitors: 0402 (20pF), 0603 (100nF), 0805 (10uF), 1206 (47uF, 100uF)
- Resistors: 0603
- LEDs: 0201
- MAX7219: SOIC-24W
- ULN2003: SOIC-16
- Switches: TL3342 tactile
- Connectors: JST PH, pin headers

Also removes accidentally committed autosave files.

Co-Authored-By: Claude Opus 4.5 <noreply@anthropic.com>
Parts:
- J9: footprint (none) -> Connector_JST:JST_PH_B4B-PH-K_1x04_P2.00mm_Vertical
Changed lines of the file:
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@@
 			)
 		)
-		(property "Footprint" ""
+		(property "Footprint" "Connector_JST:JST_PH_B4B-PH-K_1x04_P2.00mm_Vertical"
 			(at 154.94 93.98 0)
 			(effects
