File: hardware/gates.kicad_sch (KiCad schematic)
At the start: 16 parts, among them J17 GATE_T1, J18 GATE_T2, J19 GATE_T3, J20 CLK_OUT, J21 RST_OUT, U6 ULN2003

Commit message: Complete hierarchical schematic sheets and fix wiring
- Complete encoder_leds sheet with MAX7219 + 64 LEDs
- Complete ui_leds sheet with MAX7219 + 45 LEDs
- Complete buttons sheet with MCP23017 + 40 buttons
- Complete display sheet with OLED I2C connector
- Complete pots sheet with 3 potentiometers
- Complete encoders sheet with 8 rotary encoders on MCP23017
- Fix inputs sheet hierarchical labels (CLK_IN, RST_IN, SCENE_CV_IN)
- Update MCU sheet with ADC hierarchical labels
- Update root sheet with hierarchical pin connections
- Various ERC fixes and wiring corrections

Co-Authored-By: Claude Opus 4.5 <noreply@anthropic.com>
Parts:
- removed J17: GATE_T1, Connector_Audio:Jack_3.5mm_QingPu_WQP-PJ398SM_Vertical_CircularHoles, symbol Connector:AudioJack2
- removed J18: GATE_T2, Connector_Audio:Jack_3.5mm_QingPu_WQP-PJ398SM_Vertical_CircularHoles, symbol Connector:AudioJack2
- removed J19: GATE_T3, Connector_Audio:Jack_3.5mm_QingPu_WQP-PJ398SM_Vertical_CircularHoles, symbol Connector:AudioJack2
- removed J20: CLK_OUT, Connector_Audio:Jack_3.5mm_QingPu_WQP-PJ398SM_Vertical_CircularHoles, symbol Connector:AudioJack2
- removed J21: RST_OUT, Connector_Audio:Jack_3.5mm_QingPu_WQP-PJ398SM_Vertical_CircularHoles, symbol Connector:AudioJack2
- added J10: GATE_T1, symbol Connector_Audio:AudioJack2
- added J11: GATE_T2, symbol Connector_Audio:AudioJack2
- added J12: GATE_T3, symbol Connector_Audio:AudioJack2
- added J13: CLK_OUT, symbol Connector_Audio:AudioJack2
- added J14: RST_OUT, symbol Connector_Audio:AudioJack2
Connections:
- net GND: now also J10.S, J11.S, J12.S, J13.S, J14.S
- net at R26.2: now also J13.T
- net at R19.2: now also J12.T
- net at R29.2: now also J14.T
- net at R16.2: now also J10.T
- net at R17.2: now also J11.T
- no-connect marks 0 -> 2

Commit message: Assign footprints to all schematic components
SMD footprints assigned:
- Capacitors: 0402 (20pF), 0603 (100nF), 0805 (10uF), 1206 (47uF, 100uF)
- Resistors: 0603
- LEDs: 0201
- MAX7219: SOIC-24W
- ULN2003: SOIC-16
- Switches: TL3342 tactile
- Connectors: JST PH, pin headers

Also removes accidentally committed autosave files.

Co-Authored-By: Claude Opus 4.5 <noreply@anthropic.com>
Parts:
- J10, J11, J12, J13, J14: footprint (none) -> Connector_Audio:Jack_3.5mm_QingPu_WQP-PJ398SM_Vertical_CircularHoles
- R16, R17, R18, R19, R20, R25, R26, R27, R28, R29: footprint (none) -> Resistor_SMD:R_0201_0603Metric_Pad0.64x0.40mm_HandSolder
- U6: footprint (none) -> Package_SO:SOIC-16_3.9x9.9mm_P1.27mm
Changed lines of the file:
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@@
 			)
 		)
-		(property "Footprint" ""
+		(property "Footprint" "Resistor_SMD:R_0201_0603Metric_Pad0.64x0.40mm_HandSolder"
 			(at 174.752 106.68 90)
 			(effects
@@
 			)
 		)
-		(property "Footprint" ""
+		(property "Footprint" "Connector_Audio:Jack_3.5mm_QingPu_WQP-PJ398SM_Vertical_CircularHoles"
 			(at 190.5 121.92 0)
 			(effects
@@
 			)
 		)
-		(property "Footprint" ""
+		(property "Footprint" "Resistor_SMD:R_0201_0603Metric_Pad0.64x0.40mm_HandSolder"
 			(at 188.468 82.55 90)
 			(effects
@@
 			)
 		)
-		(property "Footprint" ""
+		(property "Footprint" "Resistor_SMD:R_0201_0603Metric_Pad0.64x0.40mm_HandSolder"
 			(at 170.688 82.55 90)
 			(effects
@@
 			)
 		)
-		(property "Footprint" ""
+		(property "Footprint" "Resistor_SMD:R_0201_0603Metric_Pad0.64x0.40mm_HandSolder"
 			(at 160.782 106.68 90)
 			(effects
@@
 			)
 		)
-		(property "Footprint" ""
+		(property "Footprint" "Resistor_SMD:R_0201_0603Metric_Pad0.64x0.40mm_HandSolder"
 			(at 188.722 106.68 90)
 			(effects
@@
 			)
 		)
-		(property "Footprint" ""
+		(property "Footprint" "Connector_Audio:Jack_3.5mm_QingPu_WQP-PJ398SM_Vertical_CircularHoles"
 			(at 204.47 121.92 0)
 			(effects
@@
 			)
 		)
-		(property "Footprint" ""
+		(property "Footprint" "Package_SO:SOIC-16_3.9x9.9mm_P1.27mm"
 			(at 127 110.49 0)
 			(effects
@@
 			)
 		)
-		(property "Footprint" ""
+		(property "Footprint" "Resistor_SMD:R_0201_0603Metric_Pad0.64x0.40mm_HandSolder"
 			(at 206.248 82.55 90)
 			(effects
@@
 			)
 		)
-		(property "Footprint" ""
+		(property "Footprint" "Resistor_SMD:R_0201_0603Metric_Pad0.64x0.40mm_HandSolder"
 			(at 197.358 82.55 90)
 			(effects
@@
 			)
 		)
-		(property "Footprint" ""
+		(property "Footprint" "Resistor_SMD:R_0201_0603Metric_Pad0.64x0.40mm_HandSolder"
 			(at 179.578 82.55 90)
 			(effects
@@
 			)
 		)
-		(property "Footprint" ""
+		(property "Footprint" "Resistor_SMD:R_0201_0603Metric_Pad0.64x0.40mm_HandSolder"
 			(at 146.812 106.68 90)
 			(effects
@@
 			)
 		)
-		(property "Footprint" ""
+		(property "Footprint" "Connector_Audio:Jack_3.5mm_QingPu_WQP-PJ398SM_Vertical_CircularHoles"
 			(at 176.53 120.65 0)
 			(effects
@@
 			)
 		)
-		(property "Footprint" ""
+		(property "Footprint" "Connector_Audio:Jack_3.5mm_QingPu_WQP-PJ398SM_Vertical_CircularHoles"
 			(at 162.56 120.65 0)
 			(effects
@@
 			)
 		)
-		(property "Footprint" ""
+		(property "Footprint" "Resistor_SMD:R_0201_0603Metric_Pad0.64x0.40mm_HandSolder"
 			(at 202.692 106.68 90)
 			(effects
@@
 			)
 		)
-		(property "Footprint" ""
+		(property "Footprint" "Connector_Audio:Jack_3.5mm_QingPu_WQP-PJ398SM_Vertical_CircularHoles"
 			(at 148.59 120.65 0)
 			(effects
