File: hardware/ui.kicad_sch (KiCad schematic)
At the start: 16 parts, among them J10 OLED, SW10 RUN, SW11 MODE, SW12 SCENE_L, SW13 SCENE_R

Commit message: Assign footprints to all schematic components
SMD footprints assigned:
- Capacitors: 0402 (20pF), 0603 (100nF), 0805 (10uF), 1206 (47uF, 100uF)
- Resistors: 0603
- LEDs: 0201
- MAX7219: SOIC-24W
- ULN2003: SOIC-16
- Switches: TL3342 tactile
- Connectors: JST PH, pin headers

Also removes accidentally committed autosave files.

Co-Authored-By: Claude Opus 4.5 <noreply@anthropic.com>
Parts:
- C20: footprint (none) -> Capacitor_SMD:C_0805_2012Metric
- C21: footprint (none) -> Capacitor_SMD:C_0603_1608Metric
- D1, D2, D3, D4, D5, D6, D7, D8: footprint (none) -> LED_SMD:LED_0201_0603Metric
- J10: footprint (none) -> Connector_PinHeader_2.54mm:PinHeader_1x04_P2.54mm_Vertical
- R20: footprint (none) -> Resistor_SMD:R_0603_1608Metric
- SW10, SW11, SW12, SW13: footprint (none) -> Button_Switch_SMD:SW_SPST_TL3342
Changed lines of the file:
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@@
 			(effects (font (size 1.27 1.27)))
 		)
-		(property "Footprint" ""
+		(property "Footprint" "Connector_PinHeader_2.54mm:PinHeader_1x04_P2.54mm_Vertical"
 			(at 101.6 93.59 0)
 			(effects (font (size 1.27 1.27)) hide)
@@
 			(effects (font (size 1.27 1.27)))
 		)
-		(property "Footprint" ""
+		(property "Footprint" "Resistor_SMD:R_0603_1608Metric"
 			(at 115 165 0)
 			(effects (font (size 1.27 1.27)) hide)
@@
 			(effects (font (size 1.27 1.27)) (justify left))
 		)
-		(property "Footprint" ""
+		(property "Footprint" "Capacitor_SMD:C_0805_2012Metric"
 			(at 125 165 0)
 			(effects (font (size 1.27 1.27)) hide)
@@
 			(effects (font (size 1.27 1.27)) (justify left))
 		)
-		(property "Footprint" ""
+		(property "Footprint" "Capacitor_SMD:C_0603_1608Metric"
 			(at 135 165 0)
 			(effects (font (size 1.27 1.27)) hide)
@@
 			(effects (font (size 1.27 1.27)))
 		)
-		(property "Footprint" ""
+		(property "Footprint" "LED_SMD:LED_0201_0603Metric"
 			(at 180 148 0)
 			(effects (font (size 1.27 1.27)) hide)
@@
 			(effects (font (size 1.27 1.27)))
 		)
-		(property "Footprint" ""
+		(property "Footprint" "LED_SMD:LED_0201_0603Metric"
 			(at 195 148 0)
 			(effects (font (size 1.27 1.27)) hide)
@@
 			(effects (font (size 1.27 1.27)))
 		)
-		(property "Footprint" ""
+		(property "Footprint" "LED_SMD:LED_0201_0603Metric"
 			(at 210 148 0)
 			(effects (font (size 1.27 1.27)) hide)
@@
 			(effects (font (size 1.27 1.27)))
 		)
-		(property "Footprint" ""
+		(property "Footprint" "LED_SMD:LED_0201_0603Metric"
 			(at 225 148 0)
 			(effects (font (size 1.27 1.27)) hide)
@@
 			(effects (font (size 1.27 1.27)))
 		)
-		(property "Footprint" ""
+		(property "Footprint" "LED_SMD:LED_0201_0603Metric"
 			(at 240 148 0)
 			(effects (font (size 1.27 1.27)) hide)
@@
 			(effects (font (size 1.27 1.27)))
 		)
-		(property "Footprint" ""
+		(property "Footprint" "LED_SMD:LED_0201_0603Metric"
 			(at 255 148 0)
 			(effects (font (size 1.27 1.27)) hide)
@@
 			(effects (font (size 1.27 1.27)))
 		)
-		(property "Footprint" ""
+		(property "Footprint" "LED_SMD:LED_0201_0603Metric"
 			(at 270 148 0)
 			(effects (font (size 1.27 1.27)) hide)
@@
 			(effects (font (size 1.27 1.27)))
 		)
-		(property "Footprint" ""
+		(property "Footprint" "LED_SMD:LED_0201_0603Metric"
 			(at 285 148 0)
 			(effects (font (size 1.27 1.27)) hide)
@@
 			(effects (font (size 1.27 1.27)))
 		)
-		(property "Footprint" ""
+		(property "Footprint" "Button_Switch_SMD:SW_SPST_TL3342"
 			(at 110 250 0)
 			(effects (font (size 1.27 1.27)) hide)
@@
 			(effects (font (size 1.27 1.27)))
 		)
-		(property "Footprint" ""
+		(property "Footprint" "Button_Switch_SMD:SW_SPST_TL3342"
 			(at 135 250 0)
 			(effects (font (size 1.27 1.27)) hide)
@@
 			(effects (font (size 1.27 1.27)))
 		)
-		(property "Footprint" ""
+		(property "Footprint" "Button_Switch_SMD:SW_SPST_TL3342"
 			(at 110 270 0)
 			(effects (font (size 1.27 1.27)) hide)
@@
 			(effects (font (size 1.27 1.27)))
 		)
-		(property "Footprint" ""
+		(property "Footprint" "Button_Switch_SMD:SW_SPST_TL3342"
 			(at 135 270 0)
 			(effects (font (size 1.27 1.27)) hide)
