File: hardware/ui_leds.kicad_sch (KiCad schematic)
At the start: 52 parts, among them U8 MAX7219

Commit message: Complete hierarchical schematic sheets and fix wiring
- Complete encoder_leds sheet with MAX7219 + 64 LEDs
- Complete ui_leds sheet with MAX7219 + 45 LEDs
- Complete buttons sheet with MCP23017 + 40 buttons
- Complete display sheet with OLED I2C connector
- Complete pots sheet with 3 potentiometers
- Complete encoders sheet with 8 rotary encoders on MCP23017
- Fix inputs sheet hierarchical labels (CLK_IN, RST_IN, SCENE_CV_IN)
- Update MCU sheet with ADC hierarchical labels
- Update root sheet with hierarchical pin connections
- Various ERC fixes and wiring corrections

Co-Authored-By: Claude Opus 4.5 <noreply@anthropic.com>
Connections:
- no-connect marks 0 -> 2

Commit message: Assign footprints to all schematic components
SMD footprints assigned:
- Capacitors: 0402 (20pF), 0603 (100nF), 0805 (10uF), 1206 (47uF, 100uF)
- Resistors: 0603
- LEDs: 0201
- MAX7219: SOIC-24W
- ULN2003: SOIC-16
- Switches: TL3342 tactile
- Connectors: JST PH, pin headers

Also removes accidentally committed autosave files.

Co-Authored-By: Claude Opus 4.5 <noreply@anthropic.com>
Parts:
- C18: footprint (none) -> Capacitor_SMD:C_0805_2012Metric
- C19: footprint (none) -> Capacitor_SMD:C_0603_1608Metric
- R10: footprint (none) -> Resistor_SMD:R_0201_0603Metric_Pad0.64x0.40mm_HandSolder
- U8: footprint (none) -> Package_SO:SOIC-24W_7.5x15.4mm_P1.27mm
Changed lines of the file:
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@@
 			)
 		)
-		(property "Footprint" ""
+		(property "Footprint" "Capacitor_SMD:C_0603_1608Metric"
 			(at 76.2 63.8048 0)
 			(effects
@@
 			)
 		)
-		(property "Footprint" ""
+		(property "Footprint" "Package_SO:SOIC-24W_7.5x15.4mm_P1.27mm"
 			(at 80.01 95.25 0)
 			(effects
@@
 			)
 		)
-		(property "Footprint" ""
+		(property "Footprint" "Resistor_SMD:R_0201_0603Metric_Pad0.64x0.40mm_HandSolder"
 			(at 59.69 77.978 90)
 			(effects
@@
 			)
 		)
-		(property "Footprint" ""
+		(property "Footprint" "Capacitor_SMD:C_0805_2012Metric"
 			(at 64.77 63.8048 0)
 			(effects
